Commit message: feedback linearization and jacobian

File: two-link/two-link.urdf (robot description, URDF)
Before this commit: robot pendulum, 4 links, 3 joints
Links:
- removed link link_eef
- added link link_2, mass 0; visual cylinder length=0.5 radius=0.01
- added link link_eef1, mass 1; visual sphere radius=0.05
- added link link_eef2, mass 1; visual sphere radius=0.05
Joints:
- removed joint joint_eef
- added joint joint_2: type revolute, parent link_eef1, child link_2, origin xyz=0.0 0 0 rpy=0 0 0, axis 0 1 0, limit effort=0 velocity=0
- added joint joint_eef1: type fixed, parent link_1, child link_eef1, origin xyz=0 0 0.5 rpy=0 0 0
- added joint joint_eef2: type fixed, parent link_2, child link_eef2, origin xyz=0 0 0.5 rpy=0 0 0
